File: JetsonToESC/JetsonToESC.kicad_pcb (KiCad board)
At the start: 2 copper layers, 70 x 50 mm, 47 parts, among them J1 Conn_01x12, J2 Conn_01x02, J3 Conn_01x02, J4 Screw_Terminal_01x01, J5 Screw_Terminal_01x01, U1 ESP32-C3_SUPERMINI_TH, U2 DS18B20, U3 LMR51420XDDCR, U4 MCP23018x-x-SS, U5 ACS759ECB-200B-PFF-T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

Commit message: slight edit
Routing:
- net GND: vias 45 -> 48
Other:
- board text added: "~"
Changed lines of the file:
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@@
 		(layer "Edge.Cuts")
 	)
-	(gr_text "-"
-		(at 168.6 104.9 0)
+	(gr_text "12"
+		(at 141.5 121.5 0)
+		(layer "F.SilkS")
+		(effects
+			(font
+				(size 1 1)
+				(thickness 0.1)
+			)
+			(justify left bottom)
+		)
+	)
+	(gr_text "1"
+		(at 170.3 120.4 0)
+		(layer "F.SilkS")
+		(effects
+			(font
+				(size 1 1)
+				(thickness 0.1)
+			)
+			(justify left bottom)
+		)
+	)
+	(gr_text "OUT"
+		(at 111.1 120.9 0)
+		(layer "F.SilkS")
+		(effects
+			(font
+				(size 1 1)
+				(thickness 0.2)
+				(bold yes)
+			)
+			(justify left bottom)
+		)
+	)
+	(gr_text "IN"
+		(at 112.7 90.6 0)
+		(layer "F.SilkS")
+		(effects
+			(font
+				(size 1 1)
+				(thickness 0.2)
+				(bold yes)
+			)
+			(justify left bottom)
+		)
+	)
+	(gr_text "+ Batt\nthrough"
+		(at 124.9 94.4 0)
+		(layer "F.SilkS")
+		(effects
+			(font
+				(size 1 1)
+				(thickness 0.2)
+				(bold yes)
+			)
+			(justify left bottom)
+		)
+	)
+	(gr_text "from Batt"
+		(at 172.2 97.4 0)
+		(layer "F.SilkS")
+		(effects
+			(font
+				(size 1 1)
+				(thickness 0.2)
+				(bold yes)
+			)
+			(justify left bottom)
+		)
+	)
+	(gr_text "to ESC"
+		(at 174 109 0)
+		(layer "F.SilkS")
+		(effects
+			(font
+				(size 1 1)
+				(thickness 0.2)
+				(bold yes)
+			)
+			(justify left bottom)
+		)
+	)
+	(gr_text "JetsonToESC\nv2.0\nMar 26'"
+		(at 129.7 127.3 0)
+		(layer "F.SilkS")
+		(effects
+			(font
+				(size 1 1)
+				(thickness 0.2)
+				(bold yes)
+			)
+			(justify bottom)
+		)
+	)
+	(gr_text "to\nJetson Pannel"
+		(at 139.3 124.6 90)
+		(layer "F.SilkS")
+		(effects
+			(font
+				(size 1 1)
+				(thickness 0.2)
+				(bold yes)
+			)
+			(justify bottom)
+		)
+	)
+	(gr_text "+"
+		(at 168.4 100.2 0)
 		(layer "F.SilkS")
 		(effects
@@
 		)
 	)
-	(gr_text "+"
-		(at 168.4 100.2 0)
+	(gr_text "-"
+		(at 168.6 104.9 0)
 		(layer "F.SilkS")
 		(effects
@@
 		)
 	)
-	(gr_text "1"
-		(at 169.7 120.4 0)
-		(layer "F.SilkS")
-		(effects
-			(font
-				(size 1 1)
-				(thickness 0.1)
-			)
-			(justify left bottom)
-		)
-	)
-	(gr_text "JetsonToESC\nv2.0\nMar 26'"
-		(at 129.7 127.3 0)
-		(layer "F.SilkS")
-		(effects
-			(font
-				(size 1 1)
+	(gr_text "-"
+		(at 168.6 116.5 0)
+		(layer "F.SilkS")
+		(effects
+			(font
+				(size 2 2)
 				(thickness 0.2)
 				(bold yes)
 			)
-			(justify bottom)
-		)
-	)
-	(gr_text "12"
-		(at 141.5 121.5 0)
-		(layer "F.SilkS")
-		(effects
-			(font
-				(size 1 1)
-				(thickness 0.1)
+			(justify left bottom)
+		)
+	)
+	(gr_text "~"
+		(at 169.1 111.8 0)
+		(layer "F.SilkS")
+		(effects
+			(font
+				(size 2 2)
+				(thickness 0.2)
+				(bold yes)
 			)
 			(justify left bottom)
@@
 		)
 	)
-	(gr_text "+ Batt\nthrough"
-		(at 124.9 94.4 0)
-		(layer "F.SilkS")
-		(effects
-			(font
-				(size 1 1)
-				(thickness 0.2)
-				(bold yes)
-			)
-			(justify left bottom)
-		)
-	)
-	(gr_text "-"
-		(at 168.4 116.1 0)
-		(layer "F.SilkS")
-		(effects
-			(font
-				(size 2 2)
-				(thickness 0.2)
-				(bold yes)
-			)
-			(justify left bottom)
-		)
-	)
-	(gr_text "to ESC"
-		(at 174 109 0)
-		(layer "F.SilkS")
-		(effects
-			(font
-				(size 1 1)
-				(thickness 0.2)
-				(bold yes)
-			)
-			(justify left bottom)
-		)
-	)
-	(gr_text "OUT"
-		(at 111.1 120.9 0)
-		(layer "F.SilkS")
-		(effects
-			(font
-				(size 1 1)
-				(thickness 0.2)
-				(bold yes)
-			)
-			(justify left bottom)
-		)
-	)
-	(gr_text "IN"
-		(at 112.7 90.6 0)
-		(layer "F.SilkS")
-		(effects
-			(font
-				(size 1 1)
-				(thickness 0.2)
-				(bold yes)
-			)
-			(justify left bottom)
-		)
-	)
-	(gr_text "to\nJetson Pannel"
-		(at 139.3 124.6 90)
-		(layer "F.SilkS")
-		(effects
-			(font
-				(size 1 1)
-				(thickness 0.2)
-				(bold yes)
-			)
-			(justify bottom)
-		)
-	)
-	(gr_text "from Batt"
-		(at 172.2 97.4 0)
-		(layer "F.SilkS")
-		(effects
-			(font
-				(size 1 1)
-				(thickness 0.2)
-				(bold yes)
-			)
-			(justify left bottom)
-		)
-	)
 	(segment
 		(start 167.5 120.525)
@@
 	)
 	(via
+		(at 170 110)
+		(size 0.6)
+		(drill 0.3)
+		(layers "F.Cu" "B.Cu")
+		(free yes)
+		(net 9)
+	)
+	(via
 		(at 135 100)
 		(size 0.6)
@@
 	)
 	(via
+		(at 170 115)
+		(size 0.6)
+		(drill 0.3)
+		(layers "F.Cu" "B.Cu")
+		(free yes)
+		(net 9)
+	)
+	(via
 		(at 135 95)
 		(size 0.6)
@@
 	(via
 		(at 145 105)
+		(size 0.6)
+		(drill 0.3)
+		(layers "F.Cu" "B.Cu")
+		(free yes)
+		(net 9)
+	)
+	(via
+		(at 165 110)
 		(size 0.6)
 		(drill 0.3)
@@
 	)
 	(segment
-		(start 167.35 113.25)
-		(end 168.81 111.79)
-		(width 0.127)
+		(start 168.827247 111.872753)
+		(end 172.439312 111.872753)
+		(width 0.2)
 		(layer "F.Cu")
 		(net 14)
 	)
 	(segment
-		(start 168.81 111.79)
-		(end 172.4675 111.79)
-		(width 0.127)
+		(start 167.425 113.275)
+		(end 168.827247 111.872753)
+		(width 0.2)
 		(layer "F.Cu")
 		(net 14)
+	)
+	(segment
+		(start 167.4 113.275)
+		(end 167.425 113.275)
+		(width 0.2)
+		(layer "F.Cu")
+		(net 14)

Commit message: Changing connectors from JST to Generic male 2.54mm headers
Parts:
- J1: footprint Connector_JST:JST_EH_S12B-EH_1x12_P2.50mm_Horizontal -> Connector_PinHeader_2.54mm:PinHeader_1x12_P2.54mm_Horizontal
- J2, J3: footprint Connector_JST:JST_EH_S2B-EH_1x02_P2.50mm_Horizontal -> Connector_PinHeader_2.54mm:PinHeader_1x02_P2.54mm_Horizontal
- moved C7 7.87 mm to (174.0, 96.9)
- moved J3 3.13 mm to (169.4, 99.7), turned to 0 degrees
- moved J2 3.04 mm to (169.4, 111.9), turned to 0 degrees
- moved R1 2.16 mm to (165.7, 115.3)
- moved J1 0.13 mm to (170.1, 122.4), turned to -90 degrees
Connections:
- J2 pad 2: GNDB -> GND
Routing:
- net Net-(U6-O1): track 4.88 -> 3.23 mm
- net ESC_PWM: track 5.67 -> 4.98 mm
